Commit message: extend table to 1.2x0.8m, Franka base on table surface; update docs for multi-task IK infra
Made-with: Cursor

File: assets/objects/table_simple/model.urdf (robot description, URDF)
Before this commit: robot table_simple, 1 links, 0 joints
Links:
- link base_link: mass 15.0 -> 20.0; geometry collision box size=1.2 0.8 0.05; collision cylinder length=0.75 radius=0.025
