Commit message: refactor: unify scene creation via SceneConfig pipeline
- Remove legacy hardcoded scene path in collect_data.py

- Add per-task SceneConfig presets (pick_cube, place_cube, stack_blocks, pick_bowl)

- Add scale + name_override to ObjectPlacement for 3D-gen asset scaling

- Derive object_height dynamically from PlacedObject metadata

- Shrink block URDFs from 5cm to 4cm for backward compat

- Delete is_bowl_task/is_stack_task/is_place_task flags and CUBE_SIZE/BOWL_SIZE constants

Made-with: Cursor

File: assets/objects/block_blue/model.urdf (robot description, URDF)
Before this commit: robot block_blue, 1 links, 0 joints
Links:
- link base_link: geometry collision box size=0.04 0.04 0.04; visual box size=0.04 0.04 0.04

File: assets/objects/block_green/model.urdf (robot description, URDF)
Before this commit: robot block_green, 1 links, 0 joints
Links:
- link base_link: geometry collision box size=0.04 0.04 0.04; visual box size=0.04 0.04 0.04

File: assets/objects/block_red/model.urdf (robot description, URDF)
Before this commit: robot block_red, 1 links, 0 joints
Links:
- link base_link: geometry collision box size=0.04 0.04 0.04; visual box size=0.04 0.04 0.04
