Commit message: fix: add bowl mesh files, fix URDF visual reference (.glb -> .obj), fix asset query exact match
Made-with: Cursor

File: assets/objects/bowl_01/model.urdf (robot description, URDF)
Before this commit: robot bowl_01, 1 links, 0 joints
Links:
- link base_link: geometry collision mesh filename=collision.obj; visual mesh filename=visual.obj

File: assets/objects/bowl_02/model.urdf (robot description, URDF)
Before this commit: robot bowl_02, 1 links, 0 joints
Links:
- link base_link: geometry collision mesh filename=collision.obj; visual mesh filename=visual.obj
