Commit message: sync(internal): code through cedd423 - support-surface aware grasp floor, planned place/motion, supporter scenarios (docs/tests excluded; assets limited to two_layer_supporter)

File: assets/articraft/two_layer_supporter/model.urdf (robot description, URDF)
Before this commit: robot two_layer_supporter, 1 links, 0 joints
Links:
- link base: geometry collision box size=0.008 0.17 0.28; collision box size=0.14 0.025 0.31
