Commit message: refactor(assets): bake upright rotation and metric scale into the build files
Asset build files are now metric and +Z up, so a generated asset needs no
scale or upright annotation to be placed. The rotation and scale were baked
into the meshes, the GLB root child node, and the URDF (origins, primitives,
joint limits and axes, mass x s^3, inertia R I R^T x s^5). World-frame bounds
of every asset move by at most 0.0005 mm. The articraft fixtures' 180 deg
upright yaw was a layout choice and moved into the scenes as yaw_deg.

Baking changed the build hashes, so the upright, mesh_consistency and
gripper_fit records were re-issued; the upright records point at the human
QA record they were carried over from.

Co-authored-by: Cursor <cursoragent@cursor.com>

File: assets/articraft/drawer_cabinet/model.urdf (robot description, URDF)
Before this commit: robot drawer_cabinet, 3 links, 2 joints
Links:
- link base: mass 18 -> 6.174; geometry collision box size=0.0126 0.42 0.1575; collision box size=0.028 0.028 0.07
- link drawer: mass 1.5 -> 0.5145; geometry collision box size=0.0084 0.364 0.084; collision box size=0.0126 0.406 0.147
- link drawer_handle: mass 0.05 -> 0.01715; geometry collision box size=0.035 0.0126 0.0126; collision sphere radius=0.0175
Joints:
- joint drawer_slide: limit lower=0 upper=0.35 effort=120 velocity=1 -> lower=0 upper=0.245 effort=120 velocity=1

File: assets/objects/apple_01/model.urdf (robot description, URDF)
Before this commit: robot apple_01, 1 links, 0 joints
Links:
- link base_link: mass 0.100000 -> 0.0600677

File: assets/objects/die_01/model.urdf (robot description, URDF)
Before this commit: robot die_01, 1 links, 0 joints
Links:
- link base_link: mass 0.050000 -> 0.05

File: assets/objects/lego_02/model.urdf (robot description, URDF)
Before this commit: robot lego_02, 1 links, 0 joints
Links:
- link base_link: mass 0.040000 -> 0.04

File: assets/objects/mug_02/model.urdf (robot description, URDF)
Before this commit: robot mug_02, 1 links, 0 joints
Links:
- link base_link: mass 0.250000 -> 0.0768867
